File: ver3/mystery_box-v3.kicad_pcb (KiCad board)
At the start: 2 copper layers, 136 x 100 mm, 42 parts, among them J10 Screw_Terminal_01x02, J11 Screw_Terminal_01x02, J12 Screw_Terminal_01x02, J13 Screw_Terminal_01x02, J14 Screw_Terminal_01x02, J15 Screw_Terminal_01x02, J16 Screw_Terminal_01x02, J17 Screw_Terminal_01x02, J18 Barrel_Jack_MountingPin, J20 rj45-CC-X2-Aliexpress, J4 Screw_Terminal_01x02, J8 Screw_Terminal_01x02, J9 Screw_Terminal_01x02, Q1 IRLZ44N, Q2 IRLZ44N, Q3 IRLZ44N, U2 MAX485E

Commit message: smart switch
Parts:
- removed F1, F2, F3, F4: Fuse, eigene_footprints:FUSE SPACIGER SPACER
- removed J4: Screw_Terminal_01x02, TerminalBlock:TerminalBlock_MaiXu_MX126-5.0-02P_1x02_P5.00mm
- removed R10, R6, R8: 100K, Resistor_THT:R_Axial_DIN0207_L6.3mm_D2.5mm_P10.16mm_Horizontal
- removed R4, R5, R7, R9: 330K, Resistor_THT:R_Axial_DIN0207_L6.3mm_D2.5mm_P10.16mm_Horizontal
- added R3: R100K, Resistor_THT:R_Axial_DIN0207_L6.3mm_D2.5mm_P10.16mm_Horizontal, F.Cu at (116.8, 78.0)
- added U3: ~, Package_SO:SOIC-8_3.9x4.9mm_P1.27mm, F.Cu at (119.5, 83.4)
- R3: value 100K -> R100K
Connections:
- D2 pad 1: Net-(D2-K) -> Net-(D1-K)
- D3 pad 1: Net-(D3-K) -> Net-(D1-K)
- J10 pad 2: Net-(J10-Pin_2) -> Net-(D1-K)
- J11 pad 2: Net-(J10-Pin_2) -> Net-(D1-K)
- J12 pad 2: Net-(J10-Pin_2) -> Net-(D1-K)
- J13 pad 2: Net-(J10-Pin_2) -> Net-(D1-K)
- J14 pad 2: Net-(J10-Pin_2) -> Net-(D1-K)
- J15 pad 2: Net-(J10-Pin_2) -> VCC 12V
- J16 pad 2: Net-(J10-Pin_2) -> VCC 12V
- J17 pad 2: Net-(J10-Pin_2) -> VCC 12V
- J8 pad 2: Net-(J10-Pin_2) -> Net-(D1-K)
- J9 pad 2: Net-(J10-Pin_2) -> Net-(D1-K)
- R3 pad 1: GND -> VCC 3V3
- switched_output_01 pad 1: Net-(D2-K) -> Net-(D1-K)
- switched_output_03 pad 1: Net-(D3-K) -> Net-(D1-K)

Commit message: final prototype v3
Parts:
- removed the R3 at (116.8, 78.0)
- removed the R3 at (138.9, 93.0)
- added G***: LOGO, LOGO, F.Cu at (183.5, 112.5)
- added J1: Conn_01x02_Pin, Connector_PinHeader_1.00mm:PinHeader_1x02_P1.00mm_Vertical, F.Cu at (177.5, 66.0)
- added J2: Conn_01x02_Pin, Connector_PinHeader_1.00mm:PinHeader_1x02_P1.00mm_Vertical, F.Cu at (150.5, 67.0)
- added J3: Conn_01x02_Pin, Connector_PinHeader_1.00mm:PinHeader_1x02_P1.00mm_Vertical, F.Cu at (177.5, 60.5)
- added J4: Conn_01x02_Pin, Connector_PinHeader_1.00mm:PinHeader_1x02_P1.00mm_Vertical, F.Cu at (150.5, 59.5)
- added R3: R, Resistor_THT:R_Axial_DIN0207_L6.3mm_D2.5mm_P10.16mm_Horizontal, F.Cu at (136.9, 102.5)
- added neopixel_pwr1 GND  12V: Screw_Terminal_01x02, TerminalBlock:TerminalBlock_MaiXu_MX126-5.0-02P_1x02_P5.00mm, F.Cu at (93.0, 94.5)
- moved J17 96.0 mm to (194.2, 35.0)
- moved D3 74.3 mm to (116.5, 46.4), turned to -90 degrees
- moved Q2 72.6 mm to (110.0, 79.6), turned to 180 degrees
- moved Q3 71.4 mm to (109.0, 51.1), turned to 180 degrees
- moved Q1 71.1 mm to (109.5, 65.6), turned to 180 degrees
- moved U3 70.4 mm to (189.0, 72.0)
- moved J16 60.0 mm to (206.0, 35.1)
- moved D1 51.6 mm to (116.5, 60.9), turned to -90 degrees
- moved J10 48.5 mm to (169.5, 34.9)
- moved J11 48.5 mm to (145.5, 34.9)
- moved J14 48.5 mm to (157.5, 34.9)
- moved D2 43.2 mm to (116.5, 75.9), turned to -90 degrees
- moved J12 36.8 mm to (121.4, 34.8)
- moved J8 36.8 mm to (133.4, 34.8)
- moved J15 36.0 mm to (218.0, 35.0)
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- renumbered ESP32_S1 to ESP32_S3
Connections:
- net Net-(D1-K) renamed /SW 12V
- ESP32_S3 pad 1: (no net) -> Net-(J2-Pin_1)
- ESP32_S3 pad 10: (no net) -> Net-(U3-ST)
- ESP32_S3 pad 11: (no net) -> Net-(U3-IN)
- ESP32_S3 pad 12: (no net) -> Net-(J1-Pin_1)
- ESP32_S3 pad 13: (no net) -> Net-(J1-Pin_2)
- ESP32_S3 pad 2: (no net) -> Net-(J2-Pin_2)
- ESP32_S3 pad 3: (no net) -> Net-(U2-DI)
- ESP32_S3 pad 3V3: (no net) -> unconnected-(ESP32_S3-3.3V(OUT)-Pad3V3)
- ESP32_S3 pad 4: (no net) -> Net-(U2-DE)
- ESP32_S3 pad 5: (no net) -> Net-(U1-LV3)
- ESP32_S3 pad 5V: (no net) -> Net-(J4-Pin_1)
- ESP32_S3 pad 6: (no net) -> Net-(U1-LV1)
- ESP32_S3 pad 7: (no net) -> Net-(Q2-G)
- ESP32_S3 pad 8: (no net) -> Net-(Q1-G)
- ESP32_S3 pad 9: (no net) -> Net-(Q3-G)
- ESP32_S3 pad GND: (no net) -> GND
- ESP32_S3 pad RX: (no net) -> Net-(J3-Pin_1)
- ESP32_S3 pad TX: (no net) -> Net-(J3-Pin_2)
- Q1 pad 1: Net-(ESP32_S1-8) -> Net-(Q1-G)
- Q2 pad 1: Net-(ESP32_S1-7) -> Net-(Q2-G)
- Q3 pad 1: Net-(ESP32_S1-9) -> Net-(Q3-G)
- U1 pad 1: Net-(ESP32_S1-6) -> Net-(U1-LV1)
- U1 pad 5: Net-(ESP32_S1-5) -> Net-(U1-LV3)
- U2 pad 3: Net-(ESP32_S1-4) -> Net-(U2-DE)
- U2 pad 4: Net-(ESP32_S1-3) -> Net-(U2-DI)
- U3 pad 1: Net-(ESP32_S1-11) -> Net-(U3-IN)
- U3 pad 2: Net-(ESP32_S1-10) -> Net-(U3-ST)
- U3 pad 5: VCC -> VCC 12V
- U3 pad 6: VCC -> VCC 12V
- U3 pad 7: VCC -> VCC 12V
- U3 pad 8: VCC -> VCC 12V
Routing:
- net /SW 12V: track 0.00 -> 275.3 mm
- net VCC 12V: track 0.00 -> 140.2 mm
- net Net-(Q3-G): track 0.00 -> 73.3 mm
- net Net-(Q2-G): track 0.00 -> 67.9 mm
- net Net-(Q1-G): track 0.00 -> 67.8 mm
- net Net-(U3-ST): track 0.00 -> 66.4 mm, vias 0 -> 1
- net Net-(U1-LV1): track 0.00 -> 49.5 mm, vias 0 -> 1
- net Net-(U2-DE): track 0.00 -> 48.4 mm
- net Net-(U2-DI): track 0.00 -> 48.4 mm
- net unconnected-(J20-PadSH): track 0.00 -> 46.2 mm, vias 0 -> 1
- net Net-(U1-LV3): track 0.00 -> 41.5 mm, vias 0 -> 1
- net Net-(D1-A): track 0.00 -> 29.9 mm
- net Net-(D2-A): track 0.00 -> 28.5 mm
- net Net-(D3-A): track 0.00 -> 28.1 mm
- net VCC 5V: track 0.00 -> 26.3 mm
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- added copper zone on B.Cu, net GND
- added copper zone on F.Cu, net GND
Other:
- board text added: "12V Input"
- board text added: "12V always ON"
- board text added: "12V always ON + fuse"
- board text added: "Cosmic Cable Ltd. Mysterious Prototype v3"
- board text added: "LAN"
- board text added: "POE"

Commit message: schematic with converter + footprints
Parts:
- removed 12v_input_terminal1, J10, J11, J12, J13, J14, J15, J16, J17, J8, J9, neopixel_out1, switched_output_01, switched_output_02, switched_output_03: Screw_Terminal_01x02, TerminalBlock:TerminalBlock_MaiXu_MX126-5.0-02P_1x02_P5.00mm
- removed D1, D2, D3: D, Diode_THT:D_DO-15_P10.16mm_Horizontal
- removed ESP32_S3: ~, eigene_footprints:ESP32-S3-Zero
- removed G***: LOGO, LOGO
- removed J1, J2, J3, J4: Conn_01x02_Pin, Connector_PinHeader_1.00mm:PinHeader_1x02_P1.00mm_Vertical
- removed J18: Barrel_Jack_MountingPin, eigene_footprints:CUI_PJ-050BH
- removed J20: rj45-CC-X2-Aliexpress, eigene_footprints:RJ45_X2_CC_Aliexpress
- removed Q1, Q2, Q3: IRLZ44N, Package_TO_SOT_THT:TO-220-3_Vertical
- removed R1, R2, R3: R, Resistor_THT:R_Axial_DIN0207_L6.3mm_D2.5mm_P10.16mm_Horizontal
- removed U1: ~, eigene_footprints:level_shifter
- removed U2: MAX485E, eigene_footprints:max845 modul
- removed U3: ~, Package_SO:SOIC-8_3.9x4.9mm_P1.27mm
- removed dmx_out1: DMX Out, TerminalBlock:TerminalBlock_MaiXu_MX126-5.0-03P_1x03_P5.00mm
- removed neopixel_pwr1 GND  12V: Screw_Terminal_01x02, TerminalBlock:TerminalBlock_MaiXu_MX126-5.0-02P_1x02_P5.00mm
Routing:
- net /SW 12V: track 275.3 -> 0.00 mm
- net VCC 12V: track 140.2 -> 0.00 mm
- net Net-(Q3-G): track 73.3 -> 0.00 mm
- net Net-(Q2-G): track 67.9 -> 0.00 mm
- net Net-(Q1-G): track 67.8 -> 0.00 mm
- net Net-(U3-ST): track 66.4 -> 0.00 mm, vias 1 -> 0
- net Net-(U1-LV1): track 49.5 -> 0.00 mm, vias 1 -> 0
- net Net-(U2-DE): track 48.4 -> 0.00 mm
- net Net-(U2-DI): track 48.4 -> 0.00 mm
- net unconnected-(J20-PadSH): track 46.2 -> 0.00 mm, vias 1 -> 0
- net Net-(U1-LV3): track 41.5 -> 0.00 mm, vias 1 -> 0
- net Net-(D1-A): track 29.9 -> 0.00 mm
- net Net-(D2-A): track 28.5 -> 0.00 mm
- net Net-(D3-A): track 28.1 -> 0.00 mm
- net VCC 5V: track 26.3 -> 0.00 mm
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- removed copper zone on B.Cu, net GND
- removed copper zone on F.Cu, net GND
Other:
- board outline removed
- board text removed: "12V Input"
- board text removed: "12V always ON"
- board text removed: "12V always ON + fuse"
- board text removed: "Cosmic Cable Ltd. Mysterious Prototype v3"
- board text removed: "LAN"
- board text removed: "POE"

Commit message: beginning ver3 PCB
Parts:
- added C1: 100nF, Capacitor_THT:C_Rect_L7.0mm_W2.5mm_P5.00mm, F.Cu at (-115.7, -29.2)
- added C2: 100nF, Capacitor_THT:C_Rect_L7.0mm_W2.5mm_P5.00mm, F.Cu at (-115.7, -25.1)
- added D1: D, Diode_THT:D_DO-15_P10.16mm_Horizontal, F.Cu at (-105.4, -35.5)
- added D2: D, Diode_THT:D_DO-15_P10.16mm_Horizontal, F.Cu at (-105.4, -30.4)
- added D3: D, Diode_THT:D_DO-15_P10.16mm_Horizontal, F.Cu at (-105.4, -25.2)
- added D4: 1N914, Diode_THT:D_DO-35_SOD27_P7.62mm_Horizontal, F.Cu at (-126.7, -29.4)
- added ESP32_S3: ~, eigene_footprints:ESP32-S3-Zero, F.Cu at (-127.5, -31.9)
- added GPIO13_SERIAL1: Conn_01x03_Pin, Connector_PinHeader_2.54mm:PinHeader_1x03_P2.54mm_Vertical, F.Cu at (-70.8, -60.6)
- added GPIO_CONN1: Conn_01x04_Pin, Connector_PinHeader_2.54mm:PinHeader_1x04_P2.54mm_Vertical, F.Cu at (-54.0, -33.1)
- added GPIO_T1: Screw_Terminal_01x02, TerminalBlock:TerminalBlock_MaiXu_MX126-5.0-02P_1x02_P5.00mm, F.Cu at (-124.2, -113.6)
- added GPIO_T2: Screw_Terminal_01x02, TerminalBlock:TerminalBlock_MaiXu_MX126-5.0-02P_1x02_P5.00mm, F.Cu at (-124.2, -103.5)
- added GPIO_T3: Screw_Terminal_01x02, TerminalBlock:TerminalBlock_MaiXu_MX126-5.0-02P_1x02_P5.00mm, F.Cu at (-124.2, -93.4)
- added GREEN1: LED, LED_THT:LED_D3.0mm_Horizontal_O1.27mm_Z2.0mm_Clear, F.Cu at (-50.0, -33.7)
- added J1: Screw_Terminal_01x02, TerminalBlock:TerminalBlock_MaiXu_MX126-5.0-02P_1x02_P5.00mm, F.Cu at (-124.2, -83.3)
- added J10: Screw_Terminal_01x02, TerminalBlock:TerminalBlock_MaiXu_MX126-5.0-02P_1x02_P5.00mm, F.Cu at (-111.7, -113.6)
- added J11: Screw_Terminal_01x02, TerminalBlock:TerminalBlock_MaiXu_MX126-5.0-02P_1x02_P5.00mm, F.Cu at (-111.7, -103.5)
- added J12: Screw_Terminal_01x02, TerminalBlock:TerminalBlock_MaiXu_MX126-5.0-02P_1x02_P5.00mm, F.Cu at (-111.7, -93.4)
- added J13: Screw_Terminal_01x02, TerminalBlock:TerminalBlock_MaiXu_MX126-5.0-02P_1x02_P5.00mm, F.Cu at (-111.7, -83.3)
- added J14: Screw_Terminal_01x02, TerminalBlock:TerminalBlock_MaiXu_MX126-5.0-02P_1x02_P5.00mm, F.Cu at (-111.7, -73.2)
- added J15: Screw_Terminal_01x02, TerminalBlock:TerminalBlock_MaiXu_MX126-5.0-02P_1x02_P5.00mm, F.Cu at (-111.7, -63.0)
- added J16: Screw_Terminal_01x02, TerminalBlock:TerminalBlock_MaiXu_MX126-5.0-02P_1x02_P5.00mm, F.Cu at (-99.1, -113.6)
- added J17: Screw_Terminal_01x02, TerminalBlock:TerminalBlock_MaiXu_MX126-5.0-02P_1x02_P5.00mm, F.Cu at (-99.1, -103.5)
- added J18: Barrel_Jack_MountingPin, eigene_footprints:CUI_PJ-050BH, F.Cu at (-58.5, -30.1)
- added J20: rj45-CC-X2-Aliexpress, eigene_footprints:RJ45_X2_CC_Aliexpress, F.Cu at (-71.6, -115.3)
- added J8: Screw_Terminal_01x02, TerminalBlock:TerminalBlock_MaiXu_MX126-5.0-02P_1x02_P5.00mm, F.Cu at (-124.2, -73.2)
- added J9: Screw_Terminal_01x02, TerminalBlock:TerminalBlock_MaiXu_MX126-5.0-02P_1x02_P5.00mm, F.Cu at (-124.2, -63.0)
- added JMP_24V_12V_POE1: Conn_01x03_Pin, Connector_PinHeader_2.54mm:PinHeader_1x03_P2.54mm_Vertical, F.Cu at (-66.2, -60.6)
- added JMP_5V_USB-BUCK1: Conn_01x02_Pin, Connector_PinHeader_2.54mm:PinHeader_1x02_P2.54mm_Vertical, F.Cu at (-79.9, -30.2)
- added JMP_BUCK_PWR1: Conn_01x03_Pin, Connector_PinHeader_2.54mm:PinHeader_1x03_P2.54mm_Vertical, F.Cu at (-61.6, -60.6)
- added JMP_NEO1_PWR1: Conn_01x03_Pin, Connector_PinHeader_2.54mm:PinHeader_1x03_P2.54mm_Vertical, F.Cu at (-57.0, -60.6)
- added JMP_NEO2_PWR1: Conn_01x03_Pin, Connector_PinHeader_2.54mm:PinHeader_1x03_P2.54mm_Vertical, F.Cu at (-52.4, -60.6)
- added JMP_NEO3_PWR1: Conn_01x03_Pin, Connector_PinHeader_2.54mm:PinHeader_1x03_P2.54mm_Vertical, F.Cu at (-47.8, -60.6)
- added M1: 24V-Boost-Converter, eigene_footprints:24V Boost Converter, F.Cu at (-72.3, -36.2)
- added M2: ~, eigene_footprints:5V Buck Converter, F.Cu at (-89.9, -63.6)
- added NEOPIXEL1: WS2812B, LED_SMD:LED_WS2812B_PLCC4_5.0x5.0mm_P3.2mm, F.Cu at (-103.3, -54.6)
- added NEOPIXEL2: WS2812B, LED_SMD:LED_WS2812B_PLCC4_5.0x5.0mm_P3.2mm, F.Cu at (-103.3, -48.0)
- added NEOPIXEL3: WS2812B, LED_SMD:LED_WS2812B_PLCC4_5.0x5.0mm_P3.2mm, F.Cu at (-103.3, -41.4)
- added NEO_T1: Screw_Terminal_01x03, TerminalBlock:TerminalBlock_MaiXu_MX126-5.0-03P_1x03_P5.00mm, F.Cu at (-86.6, -57.9)
- added NEO_T2: Screw_Terminal_01x03, TerminalBlock:TerminalBlock_MaiXu_MX126-5.0-03P_1x03_P5.00mm, F.Cu at (-86.6, -47.7)
- added NEO_T3: Screw_Terminal_01x03, TerminalBlock:TerminalBlock_MaiXu_MX126-5.0-03P_1x03_P5.00mm, F.Cu at (-86.6, -37.6)
- added Q1: IRLZ44N, Package_TO_SOT_THT:TO-220-3_Vertical, F.Cu at (-56.1, -78.3)
- added Q2: IRLZ44N, Package_TO_SOT_THT:TO-220-3_Vertical, F.Cu at (-56.1, -72.3)
- added Q3: IRLZ44N, Package_TO_SOT_THT:TO-220-3_Vertical, F.Cu at (-56.1, -66.4)
- added R1: 100, Resistor_THT:R_Axial_DIN0207_L6.3mm_D2.5mm_P10.16mm_Horizontal, F.Cu at (-89.0, -116.6)
- added R2: 100, Resistor_THT:R_Axial_DIN0207_L6.3mm_D2.5mm_P10.16mm_Horizontal, F.Cu at (-89.0, -112.6)
- added R3: 1k, Resistor_THT:R_Axial_DIN0207_L6.3mm_D2.5mm_P10.16mm_Horizontal, F.Cu at (-89.0, -108.5)
- added R4: 100, Resistor_THT:R_Axial_DIN0207_L6.3mm_D2.5mm_P10.16mm_Horizontal, F.Cu at (-89.0, -104.5)
- added R5: 100, Resistor_THT:R_Axial_DIN0207_L6.3mm_D2.5mm_P10.16mm_Horizontal, F.Cu at (-89.0, -100.4)
- added R6: 1k, Resistor_THT:R_Axial_DIN0207_L6.3mm_D2.5mm_P10.16mm_Horizontal, F.Cu at (-89.0, -96.4)
- added R7: 1k, Resistor_THT:R_Axial_DIN0207_L6.3mm_D2.5mm_P10.16mm_Horizontal, F.Cu at (-89.0, -92.3)
- added R8: 1k, Resistor_THT:R_Axial_DIN0207_L6.3mm_D2.5mm_P10.16mm_Horizontal, F.Cu at (-89.0, -88.3)
- added R9: 1k, Resistor_THT:R_Axial_DIN0207_L6.3mm_D2.5mm_P10.16mm_Horizontal, F.Cu at (-89.0, -84.2)
- added U3: ~, Package_SO:SOIC-8_3.9x4.9mm_P1.27mm, F.Cu at (-86.4, -29.2)
- added switched_output_01: Screw_Terminal_01x02, TerminalBlock:TerminalBlock_MaiXu_MX126-5.0-02P_1x02_P5.00mm, F.Cu at (-99.1, -93.4)
- added switched_output_02: Screw_Terminal_01x02, TerminalBlock:TerminalBlock_MaiXu_MX126-5.0-02P_1x02_P5.00mm, F.Cu at (-99.1, -83.3)
- added switched_output_03: Screw_Terminal_01x02, TerminalBlock:TerminalBlock_MaiXu_MX126-5.0-02P_1x02_P5.00mm, F.Cu at (-99.1, -73.2)

Commit message: beginning ver3 PCB
Parts:
- moved D3 224.5 mm to (65.8, 120.1)
- moved GPIO_T2 224.5 mm to (46.9, 41.8)
- moved J11 224.5 mm to (59.5, 41.8)
- moved J17 224.5 mm to (72.0, 41.8)
- moved J18 224.5 mm to (112.7, 115.1)
- moved NEOPIXEL3 224.5 mm to (67.9, 103.9)
- moved NEO_T3 224.5 mm to (84.5, 107.6)
- moved R3 224.5 mm to (82.1, 36.8)
- moved R8 224.5 mm to (82.1, 57.0)
- moved C1 224.5 mm to (55.4, 116.1)
- moved C2 224.5 mm to (55.4, 120.1)
- moved D1 224.5 mm to (65.8, 109.8)
- moved D2 224.5 mm to (65.8, 114.9)
- moved D4 224.5 mm to (44.5, 115.8)
- moved ESP32_S3 224.5 mm to (43.6, 113.3)
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
Commit message: ver3: first PCB layout
Parts:
- removed GPIO13_SERIAL1: Conn_01x03_Pin, Connector_PinHeader_2.54mm:PinHeader_1x03_P2.54mm_Vertical
- removed R5: 100, Resistor_THT:R_Axial_DIN0207_L6.3mm_D2.5mm_P10.16mm_Horizontal
- added DMX_T1: Screw_Terminal_01x03, TerminalBlock:TerminalBlock_MaiXu_MX126-5.0-03P_1x03_P5.00mm, F.Cu at (142.0, 72.5)
- added REF**: Jack_XLR_Neutrik_NC3FAAH-0_Horizontal, Connector_Audio:Jack_XLR_Neutrik_NC3FAAH-0_Horizontal, F.Cu at (150.5, 103.5)
- added SERIAL1: Conn_01x02_Pin, Connector_PinHeader_2.54mm:PinHeader_1x02_P2.54mm_Vertical, F.Cu at (187.0, 68.5)
- added U1: THVD1400D, Package_SO:SOIC-8_3.9x4.9mm_P1.27mm, F.Cu at (153.0, 79.9)
- GPIO_CONN1: value Conn_01x04_Pin -> Conn_01x03_Pin; footprint Connector_PinHeader_2.54mm:PinHeader_1x04_P2.54mm_Vertical -> Connector_PinHeader_2.54mm:PinHeader_1x03_P2.54mm_Vertical
- R6, R7, R8: value 1k -> 10k
- moved J15 209.6 mm to (269.0, 78.2), turned to 90 degrees
- moved J16 208.0 mm to (269.0, 98.2), turned to 90 degrees
- moved J17 202.4 mm to (269.0, 88.2), turned to 90 degrees
- moved J11 185.2 mm to (244.2, 29.0), turned to 180 degrees
- moved J9 185.2 mm to (224.2, 29.0), turned to 180 degrees
- moved D3 177.3 mm to (243.0, 114.1), turned to 90 degrees
- moved R9 175.2 mm to (255.5, 86.4), turned to -90 degrees
- moved J10 174.8 mm to (234.2, 29.0), turned to 180 degrees
- moved J8 172.8 mm to (214.2, 29.0), turned to 180 degrees
- moved switched_output_03 172.0 mm to (237.0, 120.8)
- moved R8 169.5 mm to (246.1, 100.0), turned to 180 degrees
- moved D2 165.8 mm to (231.5, 113.6), turned to 90 degrees
- moved switched_output_02 165.8 mm to (227.0, 120.8)
- moved switched_output_01 160.5 mm to (217.0, 120.8)
- moved J20 160.0 mm to (255.9, 64.0), turned to 90 degrees
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- renumbered D2 to D1, D1 to D2, Q2 to Q1, Q1 to Q2
Connections:
- D1 pad 2: Net-(D2-A) -> Net-(D1-A)
- D2 pad 2: Net-(D1-A) -> Net-(D2-A)
- ESP32_S3 pad 10: Net-(Q3-G) -> Net-(Q2-G)
- ESP32_S3 pad 11: Net-(U3-ST) -> Net-(Q3-G)
- ESP32_S3 pad 12: Net-(U3-IN) -> Net-(U3-ST)
- ESP32_S3 pad 13: Net-(GPIO13_SERIAL1-Pin_1) -> Net-(U3-IN)
- ESP32_S3 pad 5: Net-(NEOPIXEL1-DIN) -> Net-(U1-DE)
- ESP32_S3 pad 6: Net-(NEOPIXEL2-DIN) -> Net-(NEOPIXEL1-DIN)
- ESP32_S3 pad 7: Net-(NEOPIXEL3-DIN) -> Net-(NEOPIXEL2-DIN)
- ESP32_S3 pad 8: Net-(Q2-G) -> Net-(NEOPIXEL3-DIN)
- GPIO_T1 pad 1: Net-(GPIO_CONN1-Pin_1) -> GND
- GPIO_T1 pad 2: GND -> Net-(GPIO_CONN1-Pin_1)
- GPIO_T2 pad 1: Net-(GPIO_CONN1-Pin_3) -> GND
- GPIO_T3 pad 2: Net-(GPIO_CONN1-Pin_4) -> Net-(GPIO_CONN1-Pin_3)
- NEO_T1 pad 1: Net-(JMP_NEO1_PWR1-Pin_2) -> GND
- NEO_T1 pad 3: GND -> Net-(JMP_NEO1_PWR1-Pin_2)
- NEO_T2 pad 1: Net-(JMP_NEO2_PWR1-Pin_2) -> GND
- NEO_T2 pad 3: GND -> Net-(JMP_NEO2_PWR1-Pin_2)
- NEO_T3 pad 1: Net-(JMP_NEO3_PWR1-Pin_2) -> GND
- NEO_T3 pad 3: GND -> Net-(JMP_NEO3_PWR1-Pin_2)
- Q1 pad 1: Net-(Q2-G) -> Net-(Q1-G)
- Q1 pad 2: Net-(D2-A) -> Net-(D1-A)
- Q2 pad 1: Net-(Q1-G) -> Net-(Q2-G)
- Q2 pad 2: Net-(D1-A) -> Net-(D2-A)
- R6 pad 1: Net-(Q2-G) -> Net-(Q1-G)
- R7 pad 1: Net-(Q1-G) -> Net-(Q2-G)
- switched_output_01 pad 1: VCC 12V SW -> Net-(D1-A)
- switched_output_01 pad 2: Net-(D2-A) -> VCC 12V SW
- switched_output_02 pad 1: VCC 12V SW -> Net-(D2-A)
- switched_output_02 pad 2: Net-(D1-A) -> VCC 12V SW
- switched_output_03 pad 1: VCC 12V SW -> Net-(D3-A)
- switched_output_03 pad 2: Net-(D3-A) -> VCC 12V SW
Other:
- board outline added: 136 x 100 mm

Commit message: beginning ver3 PCB routing
Parts:
- removed REF**: Jack_XLR_Neutrik_NC3FAAH-0_Horizontal, Connector_Audio:Jack_XLR_Neutrik_NC3FAAH-0_Horizontal
- added J2: XLR3, Connector_Audio:Jack_XLR_Neutrik_NC3FAAH-0_Horizontal, F.Cu at (150.4, 104.5)
- moved JMP_BUCK_PWR1 39.0 mm to (201.0, 83.8), turned to 180 degrees
- moved R3 38.7 mm to (196.0, 50.9), turned to -90 degrees
- moved JMP_5V_USB-BUCK1 21.1 mm to (201.0, 92.6), turned to 180 degrees
- moved D4 16.8 mm to (179.3, 97.7), turned to 0 degrees
- moved U3 9.25 mm to (233.0, 74.5)
- moved U1 7.42 mm to (153.5, 72.5)
- moved M1 4.53 mm to (216.1, 54.1)
- moved JMP_24V_12V_POE1 4.27 mm to (248.0, 47.0)
- moved JMP_NEO2_PWR1 1.45 mm to (180.0, 106.6)
- moved NEOPIXEL2 1.45 mm to (187.0, 109.3)
- moved JMP_NEO3_PWR1 1.05 mm to (196.5, 106.5)
- moved C2 0.50 mm to (184.5, 44.0)
- moved NEOPIXEL3 0.35 mm to (203.0, 109.0)
- moved D1 0.25 mm to (221.0, 113.8)
- moved D2 0.25 mm to (231.5, 113.8)
Connections:
- ESP32_S3 pad 5: Net-(U1-DE) -> unconnected-(ESP32_S3-Pad5)
- U1 pad 2: unconnected-(U1-~{RE}-Pad2) -> VCC 3V3
- U1 pad 3: Net-(U1-DE) -> VCC 3V3
Routing:
- net VCC 12V SW: track 0.00 -> 293.8 mm
- net VCC 12V: track 0.00 -> 194.5 mm
- net Net-(NEOPIXEL1-DIN): track 0.00 -> 85.1 mm, vias 0 -> 1
- net Net-(NEOPIXEL3-DIN): track 0.00 -> 82.2 mm, vias 0 -> 1
- net VCC 5V USB: track 0.00 -> 72.2 mm, vias 0 -> 1
- net Net-(NEOPIXEL2-DIN): track 0.00 -> 70.7 mm, vias 0 -> 1
- net Net-(U3-IN): track 0.00 -> 57.9 mm
- net Net-(U3-ST): track 0.00 -> 55.8 mm
- net Net-(DMX_T1-Pin_1): track 0.00 -> 46.8 mm, vias 0 -> 1
- net Net-(U1-DI): track 0.00 -> 43.9 mm
- net Net-(DMX_T1-Pin_2): track 0.00 -> 37.9 mm
- net Net-(JMP_BUCK_PWR1-Pin_2): track 0.00 -> 36.6 mm
- net Net-(ESP32_S3-Pad3): track 0.00 -> 36.2 mm
- net Net-(ESP32_S3-Pad1): track 0.00 -> 26.1 mm
- net Net-(ESP32_S3-Pad2): track 0.00 -> 23.1 mm
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- added copper zone on B.Cu, net GND
- added copper zone on F.Cu, net GND

Commit message: v3: first draft finished
Parts:
- moved R8 9.94 mm to (236.1, 100.0), turned to 0 degrees
- moved JMP_NEO3_PWR1 4.85 mm to (196.6, 111.3), turned to 180 degrees
- moved JMP_NEO1_PWR1 4.62 mm to (164.6, 111.5), turned to 180 degrees
- moved JMP_NEO2_PWR1 4.59 mm to (180.0, 111.2), turned to 180 degrees
- moved JMP_BUCK_PWR1 2.27 mm to (201.2, 81.6)
- moved JMP_5V_USB-BUCK1 0.70 mm to (200.9, 93.3)
Routing:
- net Net-(Q3-G): track 0.00 -> 93.5 mm, vias 0 -> 1
- net Net-(Q2-G): track 0.00 -> 85.2 mm, vias 0 -> 1
- net Net-(Q1-G): track 0.00 -> 80.9 mm, vias 0 -> 1
- net VCC 12V SW: track 293.8 -> 356.7 mm, vias 0 -> 1
- net VCC 5V BUCK: track 13.6 -> 65.3 mm
- net VCC 3V3: track 17.4 -> 64.3 mm
- net Net-(D4-K): track 0.00 -> 45.0 mm
- net Net-(GPIO_CONN1-Pin_3): track 6.99 -> 39.9 mm
- net Net-(D2-A): track 0.00 -> 23.6 mm
- net Net-(D1-A): track 0.00 -> 23.5 mm
- net Net-(D3-A): track 0.00 -> 23.4 mm
- net Net-(JMP_NEO1_PWR1-Pin_2): track 0.00 -> 22.7 mm
- net Net-(JMP_NEO2_PWR1-Pin_2): track 0.00 -> 22.2 mm, vias 0 -> 1
- net Net-(GPIO_CONN1-Pin_2): track 6.91 -> 28.8 mm
- net Net-(JMP_NEO3_PWR1-Pin_2): track 0.00 -> 18.3 mm
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