File: ver3/mystery_box-v3.kicad_sch (KiCad schematic)
At the start: 61 parts, among them J1 Screw_Terminal_01x02, J10 Screw_Terminal_01x02, J11 Screw_Terminal_01x02, J12 Screw_Terminal_01x02, J13 Screw_Terminal_01x02, J14 Screw_Terminal_01x02, J15 Screw_Terminal_01x02, J16 Screw_Terminal_01x02, J17 Screw_Terminal_01x02, J18 Barrel_Jack_MountingPin, J20 rj45-CC-X2-Aliexpress, J3 SERIAL1, J8 Screw_Terminal_01x02, J9 Screw_Terminal_01x02, Q1 IRLZ44N, Q2 IRLZ44N, Q3 IRLZ44N, SW01 Screw_Terminal_01x02, SW02 Screw_Terminal_01x02, SW03 Screw_Terminal_01x02, U1 THVD1400D

Commit message: ver3 rev 2.0 prep for at.\tension
Parts:
- removed R5: 1k, Resistor_THT:R_Axial_DIN0207_L6.3mm_D2.5mm_P10.16mm_Horizontal, symbol Device:R
- added D5: D_Zener, Diode_THT:D_A-405_P7.62mm_Horizontal, symbol Device:D_Zener
- ESP32_S3: value ~ -> (none)
Connections:
- net VCC 12V SW: now also D5.1 (K)
- net at LED_12V_SW1.2 (A): now also D5.2 (A)
