File: ver3/mystery_box-v3.kicad_sch (KiCad schematic)
At the start: 61 parts, among them J1 Screw_Terminal_01x02, J10 Screw_Terminal_01x02, J11 Screw_Terminal_01x02, J12 Screw_Terminal_01x02, J13 Screw_Terminal_01x02, J14 Screw_Terminal_01x02, J15 Screw_Terminal_01x02, J16 Screw_Terminal_01x02, J17 Screw_Terminal_01x02, J18 Barrel_Jack_MountingPin, J20 rj45-CC-X2-Aliexpress, J3 SERIAL1, J8 Screw_Terminal_01x02, J9 Screw_Terminal_01x02, Q1 IRLZ44N, Q2 IRLZ44N, Q3 IRLZ44N, SW01 Screw_Terminal_01x02, SW02 Screw_Terminal_01x02, SW03 Screw_Terminal_01x02, U1 THVD1400D

Commit message: new 24v boost converter module
Connections:
- net GND: now also 24V-Boost-Converter1.2 (IN-); no longer 24V-Boost-Converter1.3 (IN-), 24V-Boost-Converter1.5 (OUT-), 24V-Boost-Converter1.6 (OUT-)
- net VCC 12V: no longer 24V-Boost-Converter1.2 (IN+)
- net VCC 24V: now also 24V-Boost-Converter1.3 (OUT+); no longer 24V-Boost-Converter1.7 (OUT+), 24V-Boost-Converter1.8 (OUT+)
Changed lines of the file:
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@@
 		(pin "1"
-		)
-		(pin "8"
-		)
-		(pin "6"
-		)
-		(pin "7"
-		)
-		(pin "5"
 		)
 		(instances
